Commit message: moveit2 setup successfully, can run demo launch and transform to poses

File: src/moveit_arm_package/urdf/arm.urdf.xacro (robot description, xacro)
@@ -1,12 +1,4 @@
 <?xml version="1.0"?>
 <robot name="arm_robot" xmlns:xacro="http://www.ros.org/wiki/xacro">
-    <!-- Fixed anchor so Gazebo doesn't drop the robot under gravity -->
-    <link name="world"/>
-    <joint name="world_joint" type="fixed">
-        <parent link="world"/>
-        <child link="robot_base"/>
-        <!-- z=0.05 places the bottom face of the 0.1-tall base exactly on the ground -->
-        <origin xyz="0 0 0.05" rpy="0 0 0"/>
-    </joint>
     <link name="robot_base">
         <visual>
@@ -35,5 +27,5 @@
         <collision>
             <geometry>
-                <sphere radius="0.035"/>
+                <sphere radius="0.02"/>
             </geometry>
         </collision>
@@ -61,7 +53,7 @@
         </visual>
         <collision>
-            <origin xyz="0 0 0.05" rpy="0 0 0"/>
-            <geometry>
-                <cylinder radius="0.03" length="0.1"/>
+            <origin xyz="0 0 0.04" rpy="0 0 0"/>
+            <geometry>
+                <cylinder radius="0.03" length="0.08"/>
             </geometry>
         </collision>
@@ -88,5 +80,5 @@
         <collision>
             <geometry>
-                <sphere radius="0.035"/>
+                <sphere radius="0.02"/>
             </geometry>
         </collision>
@@ -114,7 +106,7 @@
         </visual>
         <collision>
-            <origin xyz="0 0 0.15" rpy="0 0 0"/>
-            <geometry>
-                <cylinder radius="0.03" length="0.4"/>
+            <origin xyz="0 0 0.165" rpy="0 0 0"/>
+            <geometry>
+                <cylinder radius="0.03" length="0.33"/>
             </geometry>
         </collision>
@@ -141,5 +133,5 @@
         <collision>
             <geometry>
-                <sphere radius="0.035"/>
+                <sphere radius="0.02"/>
             </geometry>
         </collision>
@@ -169,5 +161,5 @@
             <origin xyz="0 0 0.15" rpy="0 0 0"/>
             <geometry>
-                <cylinder radius="0.03" length="0.35"/>
+                <cylinder radius="0.03" length="0.30"/>
             </geometry>
         </collision>
@@ -194,5 +186,5 @@
         <collision>
             <geometry>
-                <sphere radius="0.035"/>
+                <sphere radius="0.02"/>
             </geometry>
         </collision>
@@ -328,5 +320,5 @@
     <ros2_control name="GazeboSystem" type="system">
         <hardware>
-            <plugin>gazebo_ros2_control/GazeboSystem</plugin>
+            <plugin>mock_components/GenericSystem</plugin>
         </hardware>
         <joint name="shoulder_main_joint">
@@ -382,5 +374,5 @@
     <gazebo>
         <plugin name="gazebo_ros2_control" filename="libgazebo_ros2_control.so">
-            <parameters>$(find main_arm_package)/config/controllers.yaml</parameters>
+            <parameters>$(find moveit_arm_package)/config/controllers.yaml</parameters>
         </plugin>
     </gazebo>
