Commit message: fixed minor error

File: install/moveit_config/share/moveit_config/config/arm_robot.ros2_control.xacro (robot description, xacro)
@@ -8,16 +8,4 @@
                 <plugin>mock_components/GenericSystem</plugin>
             </hardware>
-            <joint name="gripper_left_finger_joint">
-                <command_interface name="position"/>
-                <state_interface name="position">
-                  <param name="initial_value">${initial_positions['gripper_left_finger_joint']}</param>
-                </state_interface>
-            </joint>
-            <joint name="gripper_right_finger_joint">
-                <command_interface name="position"/>
-                <state_interface name="position">
-                  <param name="initial_value">${initial_positions['gripper_right_finger_joint']}</param>
-                </state_interface>
-            </joint>
             <joint name="spin_main_joint">
                 <command_interface name="position"/>
