Commit message: added 2 new roll axis to the arm, now 6 axis arm, enabling moving to pose xyz and orientation

File: install/moveit_arm_package/share/moveit_arm_package/urdf/arm.urdf.xacro (robot description, xacro)
@@ -178,4 +178,56 @@
         <origin xyz="0 0 0.035" rpy="0 0 0"/>
     </joint>
+     <link name="forearm_link">
+        <visual>
+            <geometry>
+                <sphere radius="0.035"/>
+            </geometry>
+        </visual>
+        <collision>
+            <geometry>
+                <sphere radius="0.02"/>
+            </geometry>
+        </collision>
+        <inertial>
+            <mass value="0.05"/>
+            <inertia ixx="0.0000245" ixy="0" ixz="0"
+                                     iyy="0.0000245" iyz="0"
+                                                     izz="0.0000245"/>
+        </inertial>
+    </link>
+    <joint name="forearm_main_joint" type="revolute">
+        <parent link="elbow_arm"/>
+        <child link="forearm_link"/>
+        <origin xyz="0 0 0.32" rpy="0 0 0"/>
+        <axis xyz="0 0 1"/>
+        <limit lower="-3.14159" upper="3.14159" effort="10" velocity="1"/>
+        <dynamics damping="0.5" friction="0.1"/>
+    </joint>
+    <link name="forearm_arm">
+        <visual>
+            <origin xyz="0 0 0.01" rpy="0 0 0"/>
+            <geometry>
+                <cylinder radius="0.03" length="0.02"/>
+            </geometry>
+        </visual>
+        <collision>
+            <origin xyz="0 0 0.01" rpy="0 0 0"/>
+            <geometry>
+                <cylinder radius="0.03" length="0.02"/>
+            </geometry>
+        </collision>
+        <inertial>
+            <origin xyz="0 0 0.01"/>
+            <mass value="0.02"/>
+            <inertia ixx="0.0000245" ixy="0" ixz="0"
+                                     iyy="0.0000245" iyz="0"
+                                                     izz="0.0000245"/>
+        </inertial>
+    </link>
+    <joint name="forearm_arm_joint" type="fixed">
+        <parent link="forearm_link"/>
+        <child link="forearm_arm"/>
+        <origin xyz="0 0 0.035" rpy="0 0 0"/>
+    </joint>
     <link name="wrist_link">
         <visual>
@@ -197,7 +249,7 @@
     </link>
     <joint name="wrist_main_joint" type="revolute">
-        <parent link="elbow_arm"/>
+        <parent link="forearm_arm"/>
         <child link="wrist_link"/>
-        <origin xyz="0 0 0.32" rpy="0 0 0"/>
+        <origin xyz="0 0 0.02" rpy="0 0 0"/>
         <axis xyz="0 1 0"/>
         <limit lower="-2.094" upper="2.094" effort="10" velocity="1"/>
@@ -226,8 +278,11 @@
     </link>
     <!-- passive structural joint — always at 0, fixed for simulation -->
-    <joint name="wrist_arm_joint" type="fixed">
+    <joint name="wrist_arm_joint" type="revolute">
         <parent link="wrist_link"/>
         <child link="wrist_arm"/>
         <origin xyz="0 0 0.025" rpy="0 0 0"/>
+        <axis xyz="0 0 1"/>
+        <limit lower="-3.14159" upper="3.14159" effort="10" velocity="1"/>
+        <dynamics damping="0.5" friction="0.1"/>
     </joint>
     <link name="gripper_base">
@@ -347,4 +402,20 @@
         </joint>
         <joint name="spin_main_joint">
+            <command_interface name="position">
+                <param name="min">-3.14159</param>
+                <param name="max">3.14159</param>
+            </command_interface>
+            <state_interface name="position"/>
+            <state_interface name="velocity"/>
+        </joint>
+        <joint name="forearm_main_joint">
+            <command_interface name="position">
+                <param name="min">-3.14159</param>
+                <param name="max">3.14159</param>
+            </command_interface>
+            <state_interface name="position"/>
+            <state_interface name="velocity"/>
+        </joint>
+        <joint name="wrist_arm_joint">
             <command_interface name="position">
                 <param name="min">-3.14159</param>

File: install/moveit_config/share/moveit_config/config/arm_robot.ros2_control.xacro (robot description, xacro)
@@ -8,4 +8,16 @@
                 <plugin>mock_components/GenericSystem</plugin>
             </hardware>
+            <joint name="gripper_left_finger_joint">
+                <command_interface name="position"/>
+                <state_interface name="position">
+                  <param name="initial_value">${initial_positions['gripper_left_finger_joint']}</param>
+                </state_interface>
+            </joint>
+            <joint name="gripper_right_finger_joint">
+                <command_interface name="position"/>
+                <state_interface name="position">
+                  <param name="initial_value">${initial_positions['gripper_right_finger_joint']}</param>
+                </state_interface>
+            </joint>
             <joint name="spin_main_joint">
                 <command_interface name="position"/>
@@ -26,4 +38,10 @@
                 </state_interface>
             </joint>
+            <joint name="forearm_main_joint">
+                <command_interface name="position"/>
+                <state_interface name="position">
+                  <param name="initial_value">${initial_positions['forearm_main_joint']}</param>
+                </state_interface>
+            </joint>
             <joint name="wrist_main_joint">
                 <command_interface name="position"/>
@@ -32,14 +50,8 @@
                 </state_interface>
             </joint>
-            <joint name="gripper_left_finger_joint">
+            <joint name="wrist_arm_joint">
                 <command_interface name="position"/>
                 <state_interface name="position">
-                  <param name="initial_value">${initial_positions['gripper_left_finger_joint']}</param>
-                </state_interface>
-            </joint>
-            <joint name="gripper_right_finger_joint">
-                <command_interface name="position"/>
-                <state_interface name="position">
-                  <param name="initial_value">${initial_positions['gripper_right_finger_joint']}</param>
+                  <param name="initial_value">${initial_positions['wrist_arm_joint']}</param>
                 </state_interface>
             </joint>

Commit message: gazebo works with moveit (no camera)

File: install/moveit_arm_package/share/moveit_arm_package/urdf/arm.urdf.xacro (robot description, xacro)
@@ -1,4 +1,13 @@
 <?xml version="1.0"?>
 <robot name="arm_robot" xmlns:xacro="http://www.ros.org/wiki/xacro">
+    <!-- Anchor the robot to the world so it doesn't fall/collapse in Gazebo.
+         Matches the SRDF virtual_joint (fixed, parent_frame=world, child=robot_base).
+         z=0.05 lifts the 0.1m-tall base so it rests on the ground plane. -->
+    <link name="world"/>
+    <joint name="world_joint" type="fixed">
+        <parent link="world"/>
+        <child link="robot_base"/>
+        <origin xyz="0 0 0.05" rpy="0 0 0"/>
+    </joint>
     <link name="robot_base">
         <visual>
@@ -375,5 +384,6 @@
     <ros2_control name="GazeboSystem" type="system">
         <hardware>
-            <plugin>mock_components/GenericSystem</plugin>
+            <!-- Gazebo Classic 11 hardware interface (was mock_components/GenericSystem for RViz-only) -->
+            <plugin>gazebo_ros2_control/GazeboSystem</plugin>
         </hardware>
         <joint name="shoulder_main_joint">

Commit message: added camera in gazebo

File: install/moveit_arm_package/share/moveit_arm_package/urdf/arm.urdf.xacro (robot description, xacro)
@@ -10,4 +10,6 @@
         <origin xyz="0 0 0.05" rpy="0 0 0"/>
     </joint>
+    <!-- Camera on a stand, fixed in the world, looking at the arm. -->
+    <xacro:include filename="camera.xacro" />
     <link name="robot_base">
         <visual>

File: install/moveit_arm_package/share/moveit_arm_package/urdf/camera.xacro (robot description, xacro)
@@ -1,12 +1,10 @@
 <?xml version="1.0"?>
-<!-- Model name MUST stay "arm_robot" to match the MoveIt SRDF/config. -->
-<robot name="arm_robot" xmlns:xacro="http://www.ros.org/wiki/xacro">
-    <xacro:include filename="arm.urdf.xacro" />
-    <link name="world"/>
-    <joint name="world_to_arm" type="fixed">
-        <parent link="world"/>
-        <child link="robot_base"/>
-        <origin xyz="0 0 0" rpy="0 0 0"/>
-    </joint>
+<!--
+  Camera on a stand, fixed in the world, looking at the arm.
+  This is an INCLUDE FRAGMENT, not a standalone robot. It is pulled in by
+  arm.urdf.xacro via <xacro:include> and relies on the `world` link defined
+  there. Do not re-declare `world` or re-include arm.urdf.xacro here.
+-->
+<robot xmlns:xacro="http://www.ros.org/wiki/xacro">
     <link name="camera_stand">
         <visual><geometry><cylinder radius="0.02" length="1.0"/></geometry></visual>
@@ -39,4 +37,6 @@
         <origin xyz="0 0 0.5" rpy="0 0.5 3.14159"/>  <!-- tilt down, rotate to face arm -->
     </joint>
+    <!-- Optical frame: REP-103 convention (z forward, x right, y down) so the
+         published image/camera_info align with the optical axis. -->
     <link name="camera_optical_frame"/>
     <joint name="camera_optical_joint" type="fixed">
@@ -45,6 +45,9 @@
         <origin xyz="0 0 0" rpy="-1.5708 0 -1.5708"/>
     </joint>
+    <!-- Gazebo Classic camera sensor + ROS 2 plugin.
+         The published topics are <camera_name>/image_raw and
+         <camera_name>/camera_info, i.e. /camera/image_raw + /camera/camera_info. -->
     <gazebo reference="camera_link">
-        <sensor name="camera_sensor" type="camera">
+        <sensor name="camera" type="camera">
             <always_on>true</always_on>
             <update_rate>30</update_rate>
@@ -62,12 +65,8 @@
             </camera>
             <plugin name="camera_plugin" filename="libgazebo_ros_camera.so">
+                <camera_name>camera</camera_name>
                 <frame_name>camera_optical_frame</frame_name>
-                <ros>
-                    <remapping>image_raw:=/camera/image_raw</remapping>
-                    <remapping>camera_info:=/camera/camera_info</remapping>
-                </ros>
             </plugin>
         </sensor>
     </gazebo>
-    </xacro:if>
 </robot>
