Commit message: added aurco marker detection to get square position

File: install/moveit_arm_package/share/moveit_arm_package/urdf/camera.xacro (robot description, xacro)
@@ -18,5 +18,5 @@
         <parent link="world"/>
         <child link="camera_stand"/>
-        <origin xyz="0.8 0 0.5" rpy="0 0 0"/>  <!-- 0.8m in front, 0.5m high -->
+        <origin xyz="1.8 0 0.5" rpy="0 0 0"/>  <!-- 0.8m in front, 0.5m high -->
     </joint>
     <link name="camera_link">

File: src/moveit_arm_package/urdf/camera.xacro (robot description, xacro)
@@ -8,6 +8,6 @@
 <robot xmlns:xacro="http://www.ros.org/wiki/xacro">
     <link name="camera_stand">
-        <visual><geometry><cylinder radius="0.02" length="1.0"/></geometry></visual>
-        <collision><geometry><cylinder radius="0.02" length="1.0"/></geometry></collision>
+        <visual><geometry><cylinder radius="0.02" length="0.4"/></geometry></visual>
+        <collision><geometry><cylinder radius="0.02" length="0.4"/></geometry></collision>
         <inertial>
             <mass value="0.5"/>
@@ -18,5 +18,7 @@
         <parent link="world"/>
         <child link="camera_stand"/>
-        <origin xyz="0.8 0 0.5" rpy="0 0 0"/>  <!-- 0.8m in front, 0.5m high -->
+        <!-- Close-up rig: stand 0.4m tall, centered at z=0.2 so it rests on the
+             ground at x=0.6, just in front of the block at x=0.35. -->
+        <origin xyz="0.6 0 0.2" rpy="0 0 0"/>
     </joint>
     <link name="camera_link">
@@ -35,5 +37,8 @@
         <parent link="camera_stand"/>
         <child link="camera_link"/>
-        <origin xyz="0 0 0.5" rpy="0 0.5 3.14159"/>  <!-- tilt down, rotate to face arm -->
+        <!-- Camera at the top of the stand: world (0.6, 0, 0.4), ~0.48 m from the
+             block. yaw pi faces -x toward the block; pitch 0.9 rad (~52 deg)
+             tilts down to aim the optical axis at the block on the ground. -->
+        <origin xyz="0 0 0.2" rpy="0 0.9 3.14159"/>
     </joint>
     <!-- Optical frame: REP-103 convention (z forward, x right, y down) so the

Commit message: connected arm controller with vision node through topics

File: install/moveit_arm_package/share/moveit_arm_package/urdf/camera.xacro (robot description, xacro)
@@ -8,6 +8,6 @@
 <robot xmlns:xacro="http://www.ros.org/wiki/xacro">
     <link name="camera_stand">
-        <visual><geometry><cylinder radius="0.02" length="1.0"/></geometry></visual>
-        <collision><geometry><cylinder radius="0.02" length="1.0"/></geometry></collision>
+        <visual><geometry><cylinder radius="0.02" length="0.4"/></geometry></visual>
+        <collision><geometry><cylinder radius="0.02" length="0.4"/></geometry></collision>
         <inertial>
             <mass value="0.5"/>
@@ -18,5 +18,7 @@
         <parent link="world"/>
         <child link="camera_stand"/>
-        <origin xyz="1.8 0 0.5" rpy="0 0 0"/>  <!-- 0.8m in front, 0.5m high -->
+        <!-- Close-up rig: stand 0.4m tall, centered at z=0.2 so it rests on the
+             ground at x=0.6, just in front of the block at x=0.35. -->
+        <origin xyz="0.6 0 0.2" rpy="0 0 0"/>
     </joint>
     <link name="camera_link">
@@ -35,5 +37,8 @@
         <parent link="camera_stand"/>
         <child link="camera_link"/>
-        <origin xyz="0 0 0.5" rpy="0 0.5 3.14159"/>  <!-- tilt down, rotate to face arm -->
+        <!-- Camera at the top of the stand: world (0.6, 0, 0.4), ~0.48 m from the
+             block. yaw pi faces -x toward the block; pitch 0.9 rad (~52 deg)
+             tilts down to aim the optical axis at the block on the ground. -->
+        <origin xyz="0 0 0.2" rpy="0 0.9 3.14159"/>
     </joint>
     <!-- Optical frame: REP-103 convention (z forward, x right, y down) so the
@@ -45,9 +50,13 @@
         <origin xyz="0 0 0" rpy="-1.5708 0 -1.5708"/>
     </joint>
-    <!-- Gazebo Classic camera sensor + ROS 2 plugin.
-         The published topics are <camera_name>/image_raw and
-         <camera_name>/camera_info, i.e. /camera/image_raw + /camera/camera_info. -->
+    <!-- Gazebo Classic RGB-D (depth) sensor + ROS 2 plugin.
+         type="depth" makes libgazebo_ros_camera publish, all sharing
+         camera_optical_frame and the same intrinsics:
+           /camera/image_raw          (rgb)
+           /camera/depth/image_raw    (32FC1 depth in metres)
+           /camera/camera_info        (intrinsics)
+           /camera/points             (PointCloud2) -->
     <gazebo reference="camera_link">
-        <sensor name="camera" type="camera">
+        <sensor name="camera" type="depth">
             <always_on>true</always_on>
             <update_rate>30</update_rate>
@@ -67,4 +76,7 @@
                 <camera_name>camera</camera_name>
                 <frame_name>camera_optical_frame</frame_name>
+                <!-- valid depth range; readings outside come back as NaN -->
+                <min_depth>0.05</min_depth>
+                <max_depth>10.0</max_depth>
             </plugin>
         </sensor>

File: src/moveit_arm_package/urdf/camera.xacro (robot description, xacro)
@@ -50,9 +50,13 @@
         <origin xyz="0 0 0" rpy="-1.5708 0 -1.5708"/>
     </joint>
-    <!-- Gazebo Classic camera sensor + ROS 2 plugin.
-         The published topics are <camera_name>/image_raw and
-         <camera_name>/camera_info, i.e. /camera/image_raw + /camera/camera_info. -->
+    <!-- Gazebo Classic RGB-D (depth) sensor + ROS 2 plugin.
+         type="depth" makes libgazebo_ros_camera publish, all sharing
+         camera_optical_frame and the same intrinsics:
+           /camera/image_raw          (rgb)
+           /camera/depth/image_raw    (32FC1 depth in metres)
+           /camera/camera_info        (intrinsics)
+           /camera/points             (PointCloud2) -->
     <gazebo reference="camera_link">
-        <sensor name="camera" type="camera">
+        <sensor name="camera" type="depth">
             <always_on>true</always_on>
             <update_rate>30</update_rate>
@@ -72,4 +76,7 @@
                 <camera_name>camera</camera_name>
                 <frame_name>camera_optical_frame</frame_name>
+                <!-- valid depth range; readings outside come back as NaN -->
+                <min_depth>0.05</min_depth>
+                <max_depth>10.0</max_depth>
             </plugin>
         </sensor>
